Commit message: Remove deprecated files and update kinematics calculations for quaternion conversion and added some additional services

File: xacros/tool.urdf.xacro (robot description, xacro)
@@ -7,10 +7,10 @@
         <parent link="TCP"/>
         <child link="davis"/>
-	    <origin xyz="-0.10126922 0.07627988 0.11786909" rpy="-1.56978981 -0.02018286 0.04749861"/>
+	    <origin xyz="0.05 -0.063 0.105" rpy="1.5708 0 1.5708"/>
     </joint>
     <joint name="TCP_to_pressure_ft" type="fixed">
         <parent link="TCP"/>
         <child link="pressure_ft"/>
-	    <origin xyz="0.10418 0.10444 0.07405" rpy="1.54924 -0.00049 2.35537"/>
+	    <origin xyz="0.18 0. 0.105" rpy="1.5708 0 1.5708"/>
     </joint>
 </robot>
